File: stargazer/stargazer.kicad_sch (KiCad schematic)
At the start: 22 parts, among them J1 Power Terminal, J2 USB_C_Receptacle_USB2.0_14P, Q1 PMOS, U1 ESP32-C3-WROOM-02, U2 USBLC6-2SC6, U3 AP62200WU-7

Commit message: Added more sensors
Parts:
- added C10, C14, C17, C18, C9: 100n, symbol Device:C
- added C12, C4, C5, C6, C8: 1u, symbol Device:C
- added D2, D3: WS2812B, LED_SMD:LED_WS2812B_PLCC4_5.0x5.0mm_P3.2mm, symbol LED:WS2812B
- added F1: 1.5A Fuse, symbol Device:Fuse
- added SW1: SW_SPST, symbol Switch:SW_SPST
- added U3: SAM-M10Q, symbol MCU:SAM-M10Q
- added U5: MIC5504-1.8YM5, Package_TO_SOT_SMD:SOT-23-5, symbol Regulator_Linear:MIC5504-1.8YM5
- added U6: ICM-20948, symbol MCU:ICM-20948
- added U7: KX134, symbol MCU:KX134-1211
- renumbered C3 to C1, C5 to C11, C6 to C13, C7 to C15, C8 to C16, C1 to C2, C2 to C3, C4 to C7, J2 to J1, J1 to J2, R3 to R2, R2 to R3, U3 to U4
Connections:
- net +3V3: now also C17.1, C18.1, C4.1, C5.1, C6.1, C8.1, C9.1, U3.17 (VCC), U3.2 (VCC_IO), U3.3 (V_BCKP), U5.1 (VIN), U6.13 (VDD), U7.3 (IO_VDD), U7.7 (VDD)
- net GND: now also C10.2, C12.2, C14.2, C17.2, C18.2, C4.2, C5.2, C6.2, C8.2, C9.2, U3.1 (GND), U3.10 (GND), U3.11 (GND), U3.15 (GND), U3.16 (GND), U3.20 (GND), U3.4 (GND), U3.5 (GND), U3.6 (GND), U5.2 (GND), U6.11 (FSYNC), U6.18 (GND), U6.20 (RESV), U7.8 (GND), U7.9 (GND)
- net VDC: now also F1.1, SW1.2 (B); no longer C7.1, D1.1 (K), Q1.1 (D), R4.1, U4.1 (VIN)
- new net: D1.1 (K), Q1.1 (D), R4.1, SW1.1 (A)
- new net: C7.1, F1.2, U4.1 (VIN)
- new net: C14.1, U6.10 (REGOUT)
- new net: D2.2 (DOUT), D3.4 (DIN)
- new net +1V8: C10.1, C12.1, U5.5 (VOUT), U6.8 (VDDIO)
- no-connect marks 1 -> 9
Other:
- note added: "1v8 LDO + 2A Buck -> 3v3"
- note added: "LDO is only required for the ICM-20948"
- note added: "Power Mux + Switch"
- note removed: "2A Buck -> 3v3"
- note removed: "Power Mux"
- moved on the sheet: C11, C13, C15, C16, C7, D1, J2, L1, Q1, R2, R3, R4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

Commit message: Almost done stargazer
Parts:
- removed D2, D3: WS2812B, LED_SMD:LED_WS2812B_PLCC4_5.0x5.0mm_P3.2mm, symbol LED:WS2812B
- removed U5: MIC5504-1.8YM5, Package_TO_SOT_SMD:SOT-23-5, symbol Regulator_Linear:MIC5504-1.8YM5
- removed U6: ICM-20948, symbol MCU:ICM-20948
- added C19, C20, C21, C22, C25: 100n, symbol Device:C
- added C23: 1u, symbol Device:C
- added C24: 10u, symbol Device:C
- added D2: PWR_OK, symbol Device:LED
- added D4: IC_OK, symbol Device:LED
- added J3: Switch Override, symbol Connector:Screw_Terminal_01x02
- added J4: Conn_Coaxial, symbol Connector:Conn_Coaxial
- added R10, R9: 0R, symbol Device:R_US
- added R11, R13: 220, symbol Device:R_US
- added R12, R14: 4k7, symbol Device:R_US
- added R7, R8: 10k, symbol Device:R_US
- added SW2: Boot Switch, symbol Switch:SW_SPST
- added U10: ATSAMD21G18A-M, Package_DFN_QFN:QFN-48-1EP_7x7mm_P0.5mm_EP5.15x5.15mm, symbol MCU_Microchip_SAMD:ATSAMD21G18A-M
- added U5: LSM6DSO, symbol MCU:LSM6DSO
- added U6: LIS3MDL, Package_LGA:LGA-12_2x2mm_P0.5mm, symbol Sensor_Magnetic:LIS3MDL
- added U8: LPS22DF, Package_LGA:ST_HLGA-10_2x2mm_P0.5mm_LayoutBorder3x2y, symbol Sensor_Pressure:LPS22DF
- added U9: RFM95W-868S2, symbol RF_Module:RFM95W-868S2
- C10: value 100n -> 22u
- C12: value 1u -> 100n
- C8: value 1u -> 22u
- C9: value 100n -> 10u
- J2: value Power Terminal -> Battery Input
Connections:
- net +3V3: now also C12.1, C14.1, U7.1 (SDO/ADDR), U7.10 (~{CS}), C19.1, C20.1, C22.1, C23.1, C24.1, C25.1, R11.2, R7.1, R8.1, U5.1 (SDO/SA0), U5.12 (CS), U5.5 (VDDIO), U5.8 (VDD), U6.10 (~{CS}), U6.5 (Vdd), U6.6 (Vdd_IO), U6.9 (SDO/SA1), U8.1 (Vdd_IO), U8.10 (VDD), U8.5 (SA0), U8.6 (~{CS}), U9.13 (3.3V); no longer C8.1
- net D+: now also R10.1
- net D-: now also R9.1
- net GND: now also U7.4 (TRIG), C19.2, C20.2, C21.2, C22.2, C23.2, C24.2, C25.2, D2.1 (K), D4.1 (K), J4.2 (Ext), R12.2, R14.2, SW2.2 (B), U5.2 (SDx), U5.3 (SCx), U5.6 (GND), U5.7 (GND), U6.12 (GND), U6.2 (GND), U6.3 (GND), U8.3 (GND), U8.8 (GND_IO), U8.9 (GND), U9.1 (GND), U9.10 (GND), U9.8 (GND)
- net VDC: now also J3.1 (Pin_1)
- net SCL: now reaches U7.12 (SCLK/SCL)
- net SCL: now also U1.3 (IO4), U3.12 (SCL), R14.1, U5.13 (SCL), U6.1 (SCL/SPC), U8.2 (SCL)
- net SDA: now reaches U7.2 (SDI/SDA)
- net SDA: now also U1.15 (IO3), U3.9 (SDA), R12.1, U5.14 (SDA), U6.11 (SDA/SDI/SDO), U8.4 (SDA)
- net +BATT: now reaches J2.2 (Pin_2), Q1.3 (S)
- net VMUX: now reaches D1.1 (K), Q1.1 (D), R4.1, SW1.1 (A)
- net VMUX: now also J3.2 (Pin_2)
- net at C7.1, F1.2, U4.1 (VIN): now also C10.1, C8.1
- net SPI_MISO: now reaches U1.10 (IO10)
- net SPI_MISO: now also U9.2 (MISO)
- net GPS_TDX: now reaches U1.11 (RXD)
- net GPS_TDX: now also U3.13 (TXD)
- net GPS_RDX: now reaches U1.12 (TXD)
- net GPS_RDX: now also U3.14 (RXD)
- net at U1.13 (IO18): now also R9.2
- net at U1.14 (IO19): now also R10.2
- net at U1.16 (IO2): now also R8.2
- net LORA_CS: now reaches U1.17 (IO1)
- net LORA_CS: now also U9.5 (NSS)
- net LED_IC: now reaches U1.18 (IO0)
- net LED_IC: now also R13.2
- net LORA_RST: now reaches U1.4 (IO5)
- net LORA_RST: now also U9.6 (RESET)
- net SPI_CLK: now reaches U1.5 (IO6)
- net SPI_CLK: now also U9.4 (SCK)
- net SPI_MOSI: now reaches U1.6 (IO7)
- net SPI_MOSI: now also U9.3 (MOSI)
- net at U1.7 (IO8): now also R7.2
- net at U1.8 (IO9): now also SW2.1 (A)
- removed net +1V8: C10.1, C12.1
- new net: C21.1, U6.4 (C1)
- new net: J4.1 (In), U9.9 (ANT)
- new net: D4.2 (A), R13.1
- new net: U10.18 (GND), U10.35 (GND), U10.42 (GND)
- new net: D2.2 (A), R11.1
- no-connect marks 9 -> 20
Other:
- note added: "2A 3v3 Buck"
- note added: "Barometer (0x5D)"
- note added: "Battery Connector"
- note added: "Extra capacitors aren't required but some components will have very quick current draw or rely on stable voltage"
- note added: "GPS (0x84)"
- note added: "Gyro/Acc (0x6B)"
- note added: "High-G Accelerometer (0x1F)"
- note added: "IO2/IO8 High for normal boot mode"
- note added: "LoRa (SPI)"
- note added: "Magnetometer (0x1E)"
- note added: "Override incase switch deactivates during flight"
- note added: "Power Mux"
- note added: "Power Switch"
- note added: "Pull Ups"
- note added: "Status LEDs"
- note added: "USB"
- note removed: "1v8 LDO + 2A Buck -> 3v3"
- note removed: "LDO is only required for the ICM-20948"
- note removed: "Power Mux + Switch"
- note removed: "USB Mangement"
- moved on the sheet: C1, C13, C15, C16, C17, C18, C2, C3, C4, C5, C6, C7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
