File: stargazer/microcontroller.kicad_sch (KiCad schematic)
At the start: 7 parts, among them SW2 Download Mode, U2 ESP32-C3-WROOM-02

Commit message: New Layout
Parts:
- removed C7: 1u, Capacitor_SMD:C_0201_0603Metric, symbol Device:C
- removed R3: 10k, symbol Device:R_US
- removed R4: 10K, symbol Device:R_US
- added C?: 1u, Capacitor_SMD:C_0201_0603Metric, symbol Device:C
- added R?: 10k, symbol Device:R_US
- added R? (x2): 3k3, symbol Device:R_US
- SW?: renamed from SW2; value Download Mode -> swc
- renumbered C9 to C?, C8 to C?, U2 to U?
Connections:
- net BOOT_PU is gone; now on net SDA: U?.7 (IO8)
- net BOOT_SW is gone; now on net SCL: SW?.1, U?.8 (IO9)
- net +3V3: now also R?.2, R?.2, R?.2
- net GND: now also C?.2
- net SCL: now also R?.1; no longer U?.4 (IO5)
- net SDA: now also R?.1; no longer U?.3 (IO4)
- net CHIP_EN: now reaches U?.2 (EN)
- net CHIP_EN: now also C?.1, R?.1
- net D+ renamed JTAG_USB_P
- net D- renamed JTAG_USB_N
- net FLASH_CS renamed CS_LORA
- net GPS_RDX renamed TXD_GPS
- net GPS_TDX: no longer names the net of U?.11 (RXD)
- net LORA_CS renamed INT_LORA
- net LORA_INTR: no longer names the net of U?.18 (IO0)
- net LORA_RST: no longer names the net of U?.17 (IO1)
- net SPI_CLK renamed MOSI
- net SPI_MISO: no longer names the net of U?.10 (IO10)
- net SPI_MOSI renamed CS_FLASH
- new net MISO: U?.4 (IO5)
- new net SCK: U?.3 (IO4)
Other:
- note added: "When SCL is pulled low on boot the device enters DFU mode"
- moved on the sheet: C?, SW?, U?
