File: stargazer/power_mangement.kicad_sch (KiCad schematic)
At the start: 32 parts, among them J1 1984963, J2 10118193-0001LF, J3 Conn_01x02_Pin, J4 1984963, SW1 JS202011SCQN, U1 ESP32-C3-WROOM-02, U2 MCP73831-2-OT, U3 USBLC6-2SC6, U4 LM66100DCKR, U5 LM66100DCKR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

Commit message: Update
Parts:
- J1, J4: value 1984963 -> 1935161; footprint 1984963:PHOENIX_1984963 -> 1935161:PHOENIX_1935161
- R3, R4: footprint Resistor_SMD:R_0603_1608Metric -> Resistor_SMD:R_0402_1005Metric
Connections:
- net VMUX: no longer SW1.6 (C)
- net USB_N: now reaches U3.1 (I/O2)
- net USB_N: now also J2.2 (D-); no longer J2.3 (D+)
- net USB_P: now reaches U3.3 (I/O1)
- net USB_P: now also J2.3 (D+); no longer J2.2 (D-)
- net at U3.4 (I/O1): now also R3.2; no longer R4.2
- net at U3.6 (I/O2): now also R4.2; no longer R3.2
- no-connect marks 4 -> 5
Changed lines of the file:
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@@
 	)
 	(junction
-		(at 228.6 27.94)
-		(diameter 0)
-		(color 0 0 0 0)
-	)
-	(junction
-		(at 231.14 27.94)
-		(diameter 0)
-		(color 0 0 0 0)
-	)
-	(junction
 		(at 30.48 129.54)
 		(diameter 0)
@@
 	)
 	(junction
+		(at 228.6 33.02)
+		(diameter 0)
+		(color 0 0 0 0)
+	)
+	(junction
 		(at 104.14 166.37)
 		(diameter 0)
@@
 	)
 	(no_connect
+		(at 233.68 22.86)
+	)
+	(no_connect
 		(at 243.84 33.02)
 	)
@@
 	(wire
 		(pts
-			(xy 171.45 29.21) (xy 170.18 29.21)
+			(xy 228.6 33.02) (xy 233.68 33.02)
 		)
 		(stroke
@@
 	(wire
 		(pts
-			(xy 251.46 27.94) (xy 246.38 27.94)
+			(xy 171.45 29.21) (xy 170.18 29.21)
 		)
 		(stroke
@@
 	(wire
 		(pts
-			(xy 104.14 168.91) (xy 104.14 166.37)
+			(xy 251.46 27.94) (xy 246.38 27.94)
 		)
 		(stroke
@@
 	(wire
 		(pts
-			(xy 163.83 21.59) (xy 163.83 24.13)
+			(xy 104.14 168.91) (xy 104.14 166.37)
 		)
 		(stroke
@@
 	(wire
 		(pts
-			(xy 198.12 92.71) (xy 198.12 93.98)
+			(xy 163.83 21.59) (xy 163.83 24.13)
 		)
 		(stroke
@@
 	(wire
 		(pts
-			(xy 231.14 22.86) (xy 233.68 22.86)
+			(xy 198.12 92.71) (xy 198.12 93.98)
 		)
 		(stroke
@@
 	(wire
 		(pts
-			(xy 228.6 27.94) (xy 231.14 27.94)
-		)
-		(stroke
-			(width 0)
-			(type default)
-		)
-	)
-	(wire
-		(pts
-			(xy 233.68 33.02) (xy 231.14 33.02)
-		)
-		(stroke
-			(width 0)
-			(type default)
-		)
-	)
-	(wire
-		(pts
 			(xy 190.5 24.13) (xy 189.23 24.13)
 		)
@@
 	(wire
 		(pts
-			(xy 231.14 27.94) (xy 231.14 22.86)
-		)
-		(stroke
-			(width 0)
-			(type default)
-		)
-	)
-	(wire
-		(pts
 			(xy 30.48 129.54) (xy 38.1 129.54)
 		)
@@
 	(wire
 		(pts
-			(xy 228.6 38.1) (xy 228.6 27.94)
+			(xy 228.6 38.1) (xy 228.6 33.02)
 		)
 		(stroke
@@
 	(wire
 		(pts
-			(xy 231.14 33.02) (xy 231.14 27.94)
-		)
-		(stroke
-			(width 0)
-			(type default)
-		)
-	)
-	(wire
-		(pts
 			(xy 125.73 140.97) (xy 125.73 138.43)
 		)
@@
 	(wire
 		(pts
-			(xy 227.33 27.94) (xy 228.6 27.94)
+			(xy 224.79 33.02) (xy 228.6 33.02)
 		)
 		(stroke
@@
 		)
 	)
+	(label "USB_N"
+		(at 73.66 29.21 0)
+		(fields_autoplaced yes)
+		(effects
+			(font
+				(size 1.27 1.27)
+			)
+			(justify left bottom)
+		)
+	)
+	(label "USB_P"
+		(at 73.66 26.67 0)
+		(fields_autoplaced yes)
+		(effects
+			(font
+				(size 1.27 1.27)
+			)
+			(justify left bottom)
+		)
+	)
 	(global_label "SCL"
 		(shape bidirectional)
@@
 	(global_label "VMUX"
 		(shape output)
-		(at 227.33 27.94 180)
+		(at 224.79 33.02 180)
 		(fields_autoplaced yes)
 		(effects
@@
 		)
 		(property "Intersheetrefs" "${INTERSHEET_REFS}"
-			(at 219.2648 27.94 0)
+			(at 216.7248 33.02 0)
 			(effects
 				(font
@@
 			)
 		)
-		(property "Footprint" "Resistor_SMD:R_0603_1608Metric"
+		(property "Footprint" "Resistor_SMD:R_0402_1005Metric"
 			(at 116.586 30.226 90)
 			(effects
@@
 			)
 		)
-		(property "Value" "1984963"
+		(property "Value" "1935161"
 			(at 234.95 45.72 90)
 			(effects
@@
 			)
 		)
-		(property "Footprint" "1984963:PHOENIX_1984963"
+		(property "Footprint" "1935161:PHOENIX_1935161"
 			(at 240.03 43.18 0)
 			(effects
@@
 			)
 		)
-		(property "Footprint" "Resistor_SMD:R_0603_1608Metric"
+		(property "Footprint" "Resistor_SMD:R_0402_1005Metric"
 			(at 116.586 27.686 90)
 			(effects
@@
 		(dnp no)
 		(property "Reference" "SW1"
-			(at 243.84 20.32 90)
+			(at 227.33 22.86 90)
 			(effects
 				(font
@@
 		)
 		(property "Value" "JS202011SCQN"
-			(at 223.52 21.59 90)
+			(at 227.33 20.32 90)
 			(effects
 				(font
@@
 			)
 		)
-		(property "Value" "1984963"
+		(property "Value" "1935161"
 			(at 26.67 29.21 0)
 			(effects
@@
 			)
 		)
-		(property "Footprint" "1984963:PHOENIX_1984963"
+		(property "Footprint" "1935161:PHOENIX_1935161"
 			(at 26.67 26.67 0)
 			(effects

Commit message: Prerouting
Parts:
- C1, C2, C3, C4, C5, C6, C7, C8, C9: footprint Capacitor_SMD:C_0603_1608Metric -> Capacitor_SMD:C_0402_1005Metric
- R1, R10, R2, R5, R6, R7, R8: footprint Resistor_SMD:R_0603_1608Metric -> Resistor_SMD:R_0402_1005Metric

Commit message: Revision 1
Parts:
- C1, C3, C4, C6, C7, C8, C9: digikeynumber (none) -> GRM155R60J106ME05J
- C2: digikeynumber (none) -> CL05A104KA5NNNC
- C5: digikeynumber (none) -> CL05A105MQ5NNNC
- D1, D2, D4: digikeynumber (none) -> SML-LX1206SRC-TR
- J1, J4: digikeynumber (none) -> 1935161
- J2: digikeynumber (none) -> 10118193-0001LF
- R1: digikeynumber (none) -> RC0402FR-072K8L
- R10, R7, R8: digikeynumber (none) -> RC0402FR-07470RL
- R2: digikeynumber (none) -> RC0402JR-0710KL
- R3, R4: digikeynumber (none) -> RMCF0402ZT0R00
- R5, R6: digikeynumber (none) -> RC0402FR-073K3L
- SW1: digikeynumber (none) -> JS202011SCQN
- U1: digikeynumber (none) -> ESP32-C3-WROOM-02-N4
- U2: digikeynumber (none) -> MCP73831T-2ACI/OT
- U3: digikeynumber (none) -> USBLC6-2SC6
- U4, U5: digikeynumber (none) -> LM66100DCKR
- U6: digikeynumber (none) -> AP2112K-3.3TRG1

Commit message: Board Rev B WIP
Parts:
- removed R3, R4: 0, Resistor_SMD:R_0402_1005Metric, symbol Device:R_US
Connections:
- net GND: now also J2.6 (Shield)
- net JTAG_USB_N: now also U3.6 (I/O2)
- net JTAG_USB_P: now also U3.4 (I/O1)
- no-connect marks 5 -> 4
Other:
- moved on the sheet: C3, C4, C5, D1, D2, D4, J4, R10, R2, R7, R8

Commit message: Rev B schem finished
Parts:
- added R3, R4: 0, Resistor_SMD:R_0603_1608Metric, symbol Device:R_Small_US
- C1, C3, C4, C6, C7, C8, C9: footprint Capacitor_SMD:C_0402_1005Metric -> Capacitor_SMD:C_0603_1608Metric; digikeynumber GRM155R60J106ME05J -> CL10A106KQ8NNNC
- C2: footprint Capacitor_SMD:C_0402_1005Metric -> Capacitor_SMD:C_0603_1608Metric; digikeynumber CL05A104KA5NNNC -> CL10B104KO8NNWC
- C5: footprint Capacitor_SMD:C_0402_1005Metric -> Capacitor_SMD:C_0603_1608Metric; digikeynumber CL05A105MQ5NNNC -> CL10B105KP8NFNC
- R1: footprint Resistor_SMD:R_0402_1005Metric -> Resistor_SMD:R_0603_1608Metric; digikeynumber RC0402FR-072K8L -> RC0603DR-072K8L
- R2: footprint Resistor_SMD:R_0402_1005Metric -> Resistor_SMD:R_0603_1608Metric; digikeynumber RC0402JR-0710KL -> RC0603DR-0710KL
- R5, R6: footprint Resistor_SMD:R_0402_1005Metric -> Resistor_SMD:R_0603_1608Metric; digikeynumber RC0402FR-073K3L -> RC0603FR-103K3L
- R7, R8: footprint Resistor_SMD:R_0402_1005Metric -> Resistor_SMD:R_0603_1608Metric; digikeynumber RC0402FR-07470RL -> RC0603FR-13470RL
- R9: renamed from R10; footprint Resistor_SMD:R_0402_1005Metric -> Resistor_SMD:R_0603_1608Metric; digikeynumber RC0402FR-07470RL -> RC0603FR-13470RL
- U1: value ESP32-C3-WROOM-02 -> ESP32-C3-WROOM-02U-N4; footprint RF_Module:ESP32-C3-WROOM-02 -> RF_Module:ESP32-C3-WROOM-02U; digikeynumber ESP32-C3-WROOM-02-N4 -> ESP32-C3-WROOM-02U-N4
- renumbered D4 to D3
Connections:
- net JTAG_USB_N: now also R4.2; no longer U3.6 (I/O2)
- net JTAG_USB_P: now also R3.2; no longer U3.4 (I/O1)
- new net: R3.1, U3.4 (I/O1)
- new net: R4.1, U3.6 (I/O2)

Commit message: Revision B
Parts:
- removed U3: USBLC6-2SC6, Package_TO_SOT_SMD:SOT-23-6, symbol MCU:USBLC6-2SC6
Connections:
- net USB_N: now also R4.1
- net USB_P: now also R3.1
Other:
- note removed: "ESD Protection"
- moved on the sheet: R3, R4
