File: stargazer/sensors_transceivers.kicad_sch (KiCad schematic)
At the start: 40 parts, among them J3 Conn_Coaxial, J4 Micro_SD_Card, U3 SAM-M10Q, U4 RFM95W-868S2, U5 W25Q64JVSSIQ, U6 KX134, U7 LPS22DF, U8 LIS3MDL, U9 LSM6DSO

Commit message: New Layout
Parts:
- removed J3: Conn_Coaxial, symbol Connector:Conn_Coaxial
- removed J4: Micro_SD_Card, symbol Connector:Micro_SD_Card
- removed R5, R6: 4k7, symbol Device:R_US
- added J5: RFPC-SMA28-F, CON-SMA-EDGE-S:RFSOLUTIONS_CON-SMA-EDGE-S, symbol MCU:RFPC-SMA28-F
- added J6: MSD-1-A, MSD-1-A:CONN9_MSD-1_CUD, symbol MCU:MSD-1-A
- C10, C11, C23: footprint Capacitor_SMD:C_0201_0603Metric -> Capacitor_SMD:C_0603_1608Metric
- C12: renamed from C14; footprint Capacitor_SMD:C_0201_0603Metric -> Capacitor_SMD:C_0603_1608Metric
- C13: renamed from C12; footprint Capacitor_SMD:C_0201_0603Metric -> Capacitor_SMD:C_0603_1608Metric
- C14: renamed from C16; footprint Capacitor_SMD:C_0201_0603Metric -> Capacitor_SMD:C_0603_1608Metric
- C15: renamed from C13; footprint Capacitor_SMD:C_0201_0603Metric -> Capacitor_SMD:C_0603_1608Metric
- C16: renamed from C15; footprint Capacitor_SMD:C_0201_0603Metric -> Capacitor_SMD:C_0603_1608Metric
- C17: renamed from C19; footprint Capacitor_SMD:C_0201_0603Metric -> Capacitor_SMD:C_0603_1608Metric
- C18: renamed from C21; footprint Capacitor_SMD:C_0201_0603Metric -> Capacitor_SMD:C_0603_1608Metric
- C19: renamed from C20; footprint Capacitor_SMD:C_0201_0603Metric -> Capacitor_SMD:C_0603_1608Metric
- C20: renamed from C17; footprint Capacitor_SMD:C_0201_0603Metric -> Capacitor_SMD:C_0603_1608Metric
- C21: renamed from C22; footprint Capacitor_SMD:C_0201_0603Metric -> Capacitor_SMD:C_0603_1608Metric
- C22: renamed from C18; footprint Capacitor_SMD:C_0201_0603Metric -> Capacitor_SMD:C_0603_1608Metric
- C24: renamed from C26; footprint Capacitor_SMD:C_0201_0603Metric -> Capacitor_SMD:C_0603_1608Metric
- C25: renamed from C24; footprint Capacitor_SMD:C_0201_0603Metric -> Capacitor_SMD:C_0603_1608Metric
- C26: renamed from C27; footprint Capacitor_SMD:C_0201_0603Metric -> Capacitor_SMD:C_0603_1608Metric
- C27: renamed from C25; footprint Capacitor_SMD:C_0201_0603Metric -> Capacitor_SMD:C_0603_1608Metric
- R11: renamed from R7; footprint (none) -> Resistor_SMD:R_0603_1608Metric
- R12: renamed from R8; footprint (none) -> Resistor_SMD:R_0603_1608Metric
- R13: renamed from R9; footprint (none) -> Resistor_SMD:R_0603_1608Metric
- R14: renamed from R10; footprint (none) -> Resistor_SMD:R_0603_1608Metric
- R15: renamed from R11; footprint (none) -> Resistor_SMD:R_0603_1608Metric
- R16: renamed from R12; footprint (none) -> Resistor_SMD:R_0603_1608Metric
- U11: renamed from U6; footprint (none) -> Package_LGA:LGA-12_2x2mm_P0.5mm
- U13: renamed from U9; footprint (none) -> Package_LGA:LGA-14_3x2.5mm_P0.5mm_LayoutBorder3x4y
- U7: renamed from U5; value W25Q64JVSSIQ -> W25Q128JVSIQ; footprint (none) -> Package_SO:SOIC-8_5.23x5.23mm_P1.27mm
- U8: renamed from U3; footprint (none) -> RF_GPS:ublox_SAM-M8Q
- U9: renamed from U4; footprint (none) -> RF_Module:HOPERF_RFM9XW_SMD
- renumbered U7 to U10, U8 to U12
Connections:
- net +3V3: now also J6.4 (VDD)
- net GND: now also J5.2 (Ext), J6.10 (SHIELD), J6.6 (VSS)
- net at R16.1: now also J6.1 (DAT2)
- net CS_SD: now reaches R15.1
- net CS_SD: now also J6.2 (DAT3/CD)
- net at R11.1: now also J6.8 (DAT1)
- net at U9.9 (ANT): now also J5.1 (In)
- net FLASH_CS renamed CS_FLASH
- net GPS_RDX renamed TXD_GPS
- net GPS_TDX renamed RXD_GPS
- net LORA_CS renamed CS_LORA
- net LORA_INTR renamed INT_LORA
- net SPI_CLK renamed SCK
- net SCK: now also J6.5 (CLK)
- net SPI_MISO renamed MISO
- net MISO: now also J6.7 (DAT0)
- net SPI_MOSI renamed MOSI
- net MOSI: now also J6.3 (CMD)
- no-connect marks 19 -> 20
Other:
- note added: "SD Card"
- moved on the sheet: C10, C11, C12, C13, C14, C15, C16, C17, C18, C19, C20, C21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

Commit message: Update
Parts:
- added R17, R18, R19, R9: 0, Resistor_SMD:R_0402_1005Metric, symbol Device:R_US
Connections:
- net +3V3: now also R17.1, R18.2, R19.1, R9.1; no longer U10.5 (SA0), U11.1 (SDO/ADDR), U12.9 (SDO/SA1), U13.1 (SDO/SA0)
- new net: R19.2, U13.1 (SDO/SA0)
- new net: R9.2, U11.1 (SDO/ADDR)
- new net: R18.1, U10.5 (SA0)
- new net: R17.2, U12.9 (SDO/SA1)

Commit message: Prerouting
Parts:
- C10, C11, C12, C13, C14, C15, C16, C17, C18, C19, C20, C21, C22, C23, C24, C25, C26, C27: footprint Capacitor_SMD:C_0603_1608Metric -> Capacitor_SMD:C_0402_1005Metric
- R11, R12, R13, R14, R15, R16: footprint Resistor_SMD:R_0603_1608Metric -> Resistor_SMD:R_0402_1005Metric

Commit message: Revision 1
Parts:
- C10, C11, C13, C23: digikeynumber (none) -> CL05A105MQ5NNNC
- C12, C15, C17: digikeynumber (none) -> GRM155R60J106ME05J
- C14, C16, C18, C19, C20, C21, C22, C24, C25, C26, C27: digikeynumber (none) -> CL05A104KA5NNNC
- J5: value RFPC-SMA28-F -> CON-SMA-EDGE-S; digikeynumber (none) -> CON-SMA-EDGE-S
- J6: digikeynumber (none) -> MSD-1-A
- R11, R12, R13, R14, R15, R16: digikeynumber (none) -> WR04X472 JTL
- R17, R18, R19, R9: digikeynumber (none) -> RMCF0402ZT0R00
- U10: digikeynumber (none) -> LPS22DFTR
- U11: digikeynumber (none) -> KX134-1211
- U12: digikeynumber (none) -> LIS3MDLTR
- U13: digikeynumber (none) -> LSM6DSOTR
- U7: digikeynumber (none) -> W25Q128JVSIQ
- U8: digikeynumber (none) -> SAM-M10Q-00B

Commit message: Board Rev B WIP
Parts:
- removed R17, R18, R19, R9: 0, Resistor_SMD:R_0402_1005Metric, symbol Device:R_US
- added R3, R4: 4k7, Resistor_SMD:R_0402_1005Metric, symbol Device:R_US
Connections:
- net +3V3: now also U10.5 (SA0), U11.1 (SDO/ADDR), U12.9 (SDO/SA1), U13.1 (SDO/SA0), R3.1, R4.1
- net CS_FLASH: now also R4.2
- net CS_LORA: now also R3.2

Commit message: Rev B schem finished
Parts:
- added TP6: UART TXD, TestPoint:TestPoint_Pad_1.0x1.0mm, symbol Connector:TestPoint
- added TP7: UART RXD, TestPoint:TestPoint_Pad_1.0x1.0mm, symbol Connector:TestPoint
- C10, C11, C13, C23: footprint Capacitor_SMD:C_0402_1005Metric -> Capacitor_SMD:C_0603_1608Metric; digikeynumber CL05A105MQ5NNNC -> CL10B105KP8NFNC
- C12, C15, C17: footprint Capacitor_SMD:C_0402_1005Metric -> Capacitor_SMD:C_0603_1608Metric; digikeynumber GRM155R60J106ME05J -> CL10A106KQ8NNNC
- C14, C16, C18, C19, C20, C21, C22, C24, C25, C26, C27: footprint Capacitor_SMD:C_0402_1005Metric -> Capacitor_SMD:C_0603_1608Metric; digikeynumber CL05A104KA5NNNC -> CL10B104KO8NNWC
- R10: renamed from R4; footprint Resistor_SMD:R_0402_1005Metric -> Resistor_SMD:R_0603_1608Metric; digikeynumber WR04X472 JTL -> RC0603FR-074K7L
- R11: renamed from R3; footprint Resistor_SMD:R_0402_1005Metric -> Resistor_SMD:R_0603_1608Metric; digikeynumber WR04X472 JTL -> RC0603FR-074K7L
- R12: renamed from R11; footprint Resistor_SMD:R_0402_1005Metric -> Resistor_SMD:R_0603_1608Metric; digikeynumber WR04X472 JTL -> RC0603FR-074K7L
- R13: renamed from R12; footprint Resistor_SMD:R_0402_1005Metric -> Resistor_SMD:R_0603_1608Metric; digikeynumber WR04X472 JTL -> RC0603FR-074K7L
- R14: renamed from R13; footprint Resistor_SMD:R_0402_1005Metric -> Resistor_SMD:R_0603_1608Metric; digikeynumber WR04X472 JTL -> RC0603FR-074K7L
- R15: renamed from R14; footprint Resistor_SMD:R_0402_1005Metric -> Resistor_SMD:R_0603_1608Metric; digikeynumber WR04X472 JTL -> RC0603FR-074K7L
- R16: renamed from R15; footprint Resistor_SMD:R_0402_1005Metric -> Resistor_SMD:R_0603_1608Metric; digikeynumber WR04X472 JTL -> RC0603FR-074K7L
- R17: renamed from R16; footprint Resistor_SMD:R_0402_1005Metric -> Resistor_SMD:R_0603_1608Metric; digikeynumber WR04X472 JTL -> RC0603FR-074K7L
Connections:
- net RXD_GPS: now also TP7.1
- net TXD_GPS: now also TP6.1

Commit message: Revision B
Parts:
- removed TP1: SPI CLK, TestPoint:TestPoint_Pad_1.0x1.0mm, symbol Connector:TestPoint
- removed TP2: SPI MOSI, TestPoint:TestPoint_Pad_1.0x1.0mm, symbol Connector:TestPoint
- removed TP3: SPI MISO, TestPoint:TestPoint_Pad_1.0x1.0mm, symbol Connector:TestPoint
- removed TP4: I2C SDA, TestPoint:TestPoint_Pad_1.0x1.0mm, symbol Connector:TestPoint
- removed TP5: I2C SCL, TestPoint:TestPoint_Pad_1.0x1.0mm, symbol Connector:TestPoint
- removed TP6: UART TXD, TestPoint:TestPoint_Pad_1.0x1.0mm, symbol Connector:TestPoint
- removed TP7: UART RXD, TestPoint:TestPoint_Pad_1.0x1.0mm, symbol Connector:TestPoint
- U8: footprint RF_GPS:ublox_SAM-M8Q -> 1935161:ublox_SAM-M10Q
