File: stargazer/sensors_transceivers.kicad_sch (KiCad schematic)
At the start: 35 parts, among them J5 CON-SMA-EDGE-S, J6 MSD-1-A, U10 LPS22DF, U11 KX134, U12 LIS3MDL, U13 LSM6DSO, U7 W25Q128JVSIQ, U8 SAM-M10Q, U9 RFM95W-868S2

Commit message: Stargazer PCB print update
Parts:
- J5: value CON-SMA-EDGE-S -> CON-SMA-EDGE-S
Other:
- title: (none) -> Sensors & Data ICs
Changed lines of the file:
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@@
 	(generator_version "8.0")
 	(paper "USLetter")
+	(title_block
+		(title "Sensors & Data ICs")
+	)
 	(junction
 		(at 133.35 22.86)
@@
 			)
 		)
-		(property "Value" "CON-SMA-EDGE-S "
+		(property "Value" "CON-SMA-EDGE-S"
 			(at 77.47 102.87 0)
 			(effects
