File: stargazer/stargazer.kicad_pcb (KiCad board)
At the start: 2 copper layers, 70 parts, among them J1 1984963, J2 10118193-0001LF, J3 Conn_01x02_Pin, J4 1984963, J5 RFPC-SMA28-F, J6 MSD-1-A, SW1 JS202011SCQN, U1 ESP32-C3-WROOM-02, U10 LPS22DF, U11 KX134, U12 LIS3MDL, U13 LSM6DSO, U2 MCP73831-2-OT, U3 USBLC6-2SC6, U4 LM66100DCKR, U5 LM66100DCKR, U6 AP2112K-3.3, U7 W25Q128JVSIQ, U8 SAM-M10Q, U9 RFM95W-868S2

Commit message: Update
Parts:
- added H1: MountingHole, MountingHole:MountingHole_3.2mm_M3_DIN965_Pad, F.Cu at (153.5, 25.0)
- added H2: MountingHole, MountingHole:MountingHole_3.2mm_M3_DIN965_Pad, F.Cu at (153.0, 60.5)
- added H3: MountingHole, MountingHole:MountingHole_3.2mm_M3_DIN965_Pad, F.Cu at (228.0, 25.0)
- added H4: MountingHole, MountingHole:MountingHole_3.2mm_M3_DIN965_Pad, F.Cu at (228.2, 60.0)
- added R17: 0, Resistor_SMD:R_0402_1005Metric, F.Cu at (124.8, 47.5)
- added R18: 0, Resistor_SMD:R_0402_1005Metric, F.Cu at (120.8, 59.5)
- added R19: 0, Resistor_SMD:R_0402_1005Metric, F.Cu at (124.8, 27.2)
- added R9: 0, Resistor_SMD:R_0402_1005Metric, F.Cu at (119.8, 38.8)
- J1, J4: value 1984963 -> 1935161; footprint 1984963:PHOENIX_1984963 -> 1935161:PHOENIX_1935161
- R3, R4: footprint Resistor_SMD:R_0603_1608Metric -> Resistor_SMD:R_0402_1005Metric
- moved J3 111.2 mm to (219.2, 30.5), turned to 90 degrees
- moved R5 106.4 mm to (237.6, 23.6)
- moved U1 105.5 mm to (224.8, 42.0), turned to -90 degrees
- moved U11 97.4 mm to (121.7, 39.0)
- moved R6 96.7 mm to (237.7, 20.5)
- moved C5 93.9 mm to (227.0, 31.5), turned to 180 degrees
- moved U12 93.4 mm to (122.9, 47.5)
- moved C2 93.1 mm to (230.0, 31.5), turned to 180 degrees
- moved C1 92.6 mm to (230.0, 30.0), turned to 180 degrees
- moved U13 90.1 mm to (127.1, 27.5)
- moved R2 90.0 mm to (227.0, 30.0), turned to 180 degrees
- moved C9 87.4 mm to (236.0, 86.5), turned to -90 degrees
- moved C8 86.4 mm to (234.5, 86.5), turned to -90 degrees
- moved U6 85.1 mm to (231.4, 86.5)
- moved TP5 84.5 mm to (116.0, 70.5), turned to 180 degrees
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Connections:
- J2 pad 2: Net-(J2-D-) -> /Power Mangement And MCU/USB_N
- J2 pad 3: Net-(J2-D+) -> /Power Mangement And MCU/USB_P
- SW1 pad 6: VMUX -> unconnected-(SW1-C-Pad6)
- U10 pad 5: +3V3 -> Net-(U10-SA0)
- U11 pad 1: +3V3 -> Net-(U11-SDO/ADDR)
- U12 pad 9: +3V3 -> Net-(U12-SDO/SA1)
- U13 pad 1: +3V3 -> Net-(U13-SDO/SA0)
- U3 pad 1: Net-(J2-D+) -> /Power Mangement And MCU/USB_N
- U3 pad 3: Net-(J2-D-) -> /Power Mangement And MCU/USB_P
- U3 pad 4: Net-(R4-Pad2) -> Net-(R3-Pad2)
- U3 pad 6: Net-(R3-Pad2) -> Net-(R4-Pad2)
Other:
- board outline added: 82.5 x 43 mm
- board text added: "BATTERY (GND)"
- board text added: "CHRG"
- board text added: "MCU"
- board text added: "PWR"
- board text added: "PWR OVERRIDE"
- board text added: "STATUS LEDS"

Commit message: Prerouting
Parts:
- added G***: LOGO, LOGO, B.Cu at (166.4, 94.7)
- added G***: LOGO, LOGO, B.Cu at (177.5, 94.7)
- added G***: LOGO, LOGO, B.Cu at (134.2, 94.7)
- C1, C10, C11, C12, C13, C14, C15, C16, C17, C18, C19, C2, C20, C21, C22, C23, C24, C25, C26, C27, C3, C4, C5, C6, C7, C8, C9: footprint Capacitor_SMD:C_0603_1608Metric -> Capacitor_SMD:C_0402_1005Metric
- R1, R10, R11, R12, R13, R14, R15, R16, R2, R5, R6, R7, R8: footprint Resistor_SMD:R_0603_1608Metric -> Resistor_SMD:R_0402_1005Metric
- moved R6 115.5 mm to (153.4, 99.5)
- moved R5 112.6 mm to (153.4, 98.4)
- moved R11 112.6 mm to (146.4, 92.0)
- moved R12 112.0 mm to (145.2, 92.0)
- moved R13 111.5 mm to (144.0, 92.0)
- moved C17 110.9 mm to (141.6, 92.0), turned to -90 degrees
- moved J6 110.0 mm to (140.5, 81.9)
- moved C19 109.7 mm to (142.8, 92.0), turned to -90 degrees
- moved R14 108.6 mm to (140.4, 92.0)
- moved D1 108.0 mm to (123.9, 111.5)
- moved D2 108.0 mm to (118.9, 111.5)
- moved D4 108.0 mm to (128.5, 111.4)
- moved R15 108.0 mm to (139.2, 92.0)
- moved R10 107.9 mm to (126.8, 111.9), turned to 90 degrees
- moved R7 107.9 mm to (122.2, 111.9), turned to 90 degrees
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Routing:
- net SCL: track 0.00 -> 37.5 mm
- net SDA: track 0.00 -> 31.4 mm
- net +3V3: track 0.00 -> 30.2 mm
- net TXD_GPS: track 0.00 -> 25.5 mm, vias 0 -> 2
- net RXD_GPS: track 0.00 -> 22.9 mm, vias 0 -> 2
- net VBUS: track 0.00 -> 19.9 mm
- net GND: track 0.00 -> 18.1 mm, vias 0 -> 2
- net JTAG_USB_N: track 0.00 -> 5.59 mm
- net JTAG_USB_P: track 0.00 -> 5.55 mm
- net +BATT: track 0.00 -> 3.54 mm
- net CHIP_EN: track 0.00 -> 2.83 mm
- net /Power Mangement And MCU/USB_P: track 0.00 -> 2.70 mm
- net /Power Mangement And MCU/USB_N: track 0.00 -> 2.70 mm
- net Net-(U2-PROG): track 0.00 -> 1.60 mm
- net Net-(R4-Pad2): track 0.00 -> 1.44 mm
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- added copper zone on B.Cu, net GND
- added copper zone on F.Cu, net GND
Other:
- board size 82.5 x 43 mm -> 72 x 40.8 mm
- rule pad_to_mask_clearance: 0 -> 0.038
- board text added: "BACKUP FLASH"
- board text added: "BATT (GND)"
- board text added: "BOOT"
- board text added: "JLCJLCJLCJLC"
- board text added: "Nick Coombe (www.coombe.lol) Rev. A"
- board text added: "OVERRIDE"
- board text added: "PCB3D_BR_main"
- board text added: "PCB3D_TL_main"
- board text removed: "BATTERY (GND)"
- board text removed: "PWR OVERRIDE"

Commit message: Revision 1
Parts:
- moved R9 13.2 mm to (137.4, 99.9), turned to 0 degrees
- moved C22 12.9 mm to (136.2, 103.7), turned to 0 degrees
- moved U11 12.2 mm to (137.2, 101.8), turned to -90 degrees
- moved C20 10.1 mm to (138.2, 103.7), turned to 180 degrees
- moved C18 9.55 mm to (145.3, 94.1), turned to 0 degrees
- moved C21 9.32 mm to (143.6, 95.3), turned to 90 degrees
- moved C23 7.25 mm to (146.8, 100.0)
- moved C25 7.25 mm to (145.2, 103.7)
- moved C27 7.25 mm to (143.6, 102.1)
- moved U12 7.25 mm to (145.6, 101.8)
- moved R17 7.25 mm to (147.4, 101.5)
- moved TP5 7.11 mm to (154.5, 94.5)
- moved U10 5.95 mm to (145.4, 96.0), turned to 0 degrees
- moved C24 5.00 mm to (135.5, 98.3), turned to 180 degrees
- moved R18 4.79 mm to (147.2, 96.3), turned to 90 degrees
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- renumbered G*** to logo, G*** to winsatlogo
Routing:
- net +3V3: track 30.2 -> 242.3 mm, vias 0 -> 4
- net SCK: track 0.00 -> 88.2 mm, vias 0 -> 3
- net MOSI: track 0.00 -> 87.8 mm, vias 0 -> 3
- net MISO: track 0.00 -> 87.4 mm, vias 0 -> 3
- net LORA_RST: track 0.00 -> 87.4 mm, vias 0 -> 2
- net INT_LORA: track 0.00 -> 66.6 mm, vias 0 -> 2
- net CS_SD: track 0.00 -> 66.3 mm, vias 0 -> 2
- net CS_LORA: track 0.00 -> 66.2 mm, vias 0 -> 2
- net LED_STATUS: track 0.00 -> 58.0 mm, vias 0 -> 2
- net CS_FLASH: track 0.00 -> 54.1 mm, vias 0 -> 2
- net VDC: track 0.00 -> 43.0 mm
- net BATT_STAT: track 0.00 -> 42.8 mm
- net VMUX: track 0.00 -> 35.2 mm
- net SCL: track 37.5 -> 63.9 mm, vias 0 -> 4
- net SDA: track 31.4 -> 57.8 mm, vias 0 -> 2
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Other:
- board text added: "Nick Coombe (www.quizque.ca) Rev. A"
- board text removed: "Nick Coombe (www.coombe.lol) Rev. A"

Commit message: Board Rev B WIP
Parts:
- J5: value RFPC-SMA28-F -> CON-SMA-EDGE-S
Connections:
- J2 pad 6: unconnected-(J2-Shield-Pad6) -> GND
Routing:
- net VMUX: track 35.2 -> 38.2 mm
- net SCK: track 88.2 -> 89.0 mm
- net GND: vias 81 -> 106
- net (no net): vias 25 -> 0

Commit message: Revision B
Parts:
- removed D4: SML-LX1206SRC-TR, LED_SMD:LED_0805_2012Metric
- removed R18, R19: 0, Resistor_SMD:R_0402_1005Metric
- removed TP1: SPI CLK, TestPoint:TestPoint_Pad_1.0x1.0mm
- removed TP2: SPI MOSI, TestPoint:TestPoint_Pad_1.0x1.0mm
- removed TP3: SPI MISO, TestPoint:TestPoint_Pad_1.0x1.0mm
- removed TP4: I2C SDA, TestPoint:TestPoint_Pad_1.0x1.0mm
- removed TP5: I2C SCL, TestPoint:TestPoint_Pad_1.0x1.0mm
- removed U3: USBLC6-2SC6, Package_TO_SOT_SMD:SOT-23-6
- added D3: SML-LX1206SRC-TR, LED_SMD:LED_0805_2012Metric, F.Cu at (119.5, 111.2)
- C1, C10, C11, C12, C13, C14, C15, C16, C17, C18, C19, C2, C20, C21, C22, C23, C24, C25, C26, C27, C3, C4, C5, C6, C7, C8, C9: footprint Capacitor_SMD:C_0402_1005Metric -> Capacitor_SMD:C_0603_1608Metric
- R1, R11, R12, R13, R14, R15, R16, R2, R3, R4, R5, R6, R7, R8: footprint Resistor_SMD:R_0402_1005Metric -> Resistor_SMD:R_0603_1608Metric
- R10: value 470 -> 4k7; footprint Resistor_SMD:R_0402_1005Metric -> Resistor_SMD:R_0603_1608Metric
- R17: value 0 -> 4k7; footprint Resistor_SMD:R_0402_1005Metric -> Resistor_SMD:R_0603_1608Metric
- R9: value 0 -> 470; footprint Resistor_SMD:R_0402_1005Metric -> Resistor_SMD:R_0603_1608Metric
- U1: value ESP32-C3-WROOM-02 -> ESP32-C3-WROOM-02U-N4; footprint RF_Module:ESP32-C3-WROOM-02 -> RF_Module:ESP32-C3-WROOM-02U
- U8: footprint RF_GPS:ublox_SAM-M8Q -> 1935161:ublox_SAM-M10Q
- moved R10 30.3 mm to (128.6, 81.6), turned to -90 degrees
- moved R9 22.9 mm to (117.5, 111.2), turned to 90 degrees
- moved R17 14.5 mm to (136.2, 92.4)
- moved R11 13.6 mm to (133.2, 95.2)
- moved C14 11.7 mm to (117.4, 81.4)
- moved D2 10.2 mm to (129.0, 111.3)
- moved R8 9.82 mm to (127.0, 111.3)
- moved C6 6.03 mm to (164.8, 94.2), turned to 180 degrees
- moved R3 4.85 mm to (174.2, 107.2), turned to 90 degrees
- moved R4 4.77 mm to (172.2, 107.2), turned to 90 degrees
- moved R1 4.61 mm to (151.8, 103.3), turned to -90 degrees
- moved C26 4.41 mm to (138.6, 97.6), turned to 90 degrees
- moved R14 3.79 mm to (144.2, 92.4)
- moved C18 3.16 mm to (147.0, 96.8), turned to 90 degrees
- moved C24 3.14 mm to (136.0, 95.2)
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Connections:
- R10 pad 1: Net-(D4-K) -> +3V3
- R10 pad 2: GND -> CS_FLASH
- R11 pad 1: Net-(J6-DAT1) -> +3V3
- R11 pad 2: +3V3 -> CS_LORA
- R12 pad 1: MISO -> Net-(J6-DAT1)
- R13 pad 1: SCK -> MISO
- R14 pad 1: MOSI -> SCK
- R15 pad 1: CS_SD -> MOSI
- R16 pad 1: Net-(J6-DAT2) -> CS_SD
- R17 pad 1: +3V3 -> Net-(J6-DAT2)
- R17 pad 2: Net-(U12-SDO/SA1) -> +3V3
- R3 pad 1: JTAG_USB_P -> /Power Mangement And MCU/USB_P
- R3 pad 2: Net-(R3-Pad2) -> JTAG_USB_P
- R4 pad 1: JTAG_USB_N -> /Power Mangement And MCU/USB_N
- R4 pad 2: Net-(R4-Pad2) -> JTAG_USB_N
- R9 pad 1: +3V3 -> Net-(D3-K)
- R9 pad 2: Net-(U11-SDO/ADDR) -> GND
- U10 pad 5: Net-(U10-SA0) -> +3V3
- U11 pad 1: Net-(U11-SDO/ADDR) -> +3V3
- U12 pad 9: Net-(U12-SDO/SA1) -> +3V3
- U13 pad 1: Net-(U13-SDO/SA0) -> +3V3
Routing:
- net LORA_RST: track 87.4 -> 57.5 mm
- net GND: track 24.5 -> 51.9 mm, vias 106 -> 79
- net CS_SD: track 66.3 -> 39.1 mm, vias 2 -> 4
- net INT_LORA: track 66.6 -> 80.5 mm
- net +3V3: track 242.3 -> 230.2 mm, vias 4 -> 2
- net LED_STATUS: track 58.0 -> 69.5 mm
- net BATT_STAT: track 42.8 -> 32.2 mm
- net SDA: track 57.8 -> 48.7 mm, vias 2 -> 4
- net SCK: track 89.0 -> 97.6 mm, vias 3 -> 5
- net CS_LORA: track 66.2 -> 74.3 mm
- net MOSI: track 87.8 -> 94.8 mm
- net VDC: track 43.0 -> 48.3 mm
- net JTAG_USB_N: track 5.59 -> 2.28 mm
- net JTAG_USB_P: track 5.55 -> 2.28 mm
- net /Power Mangement And MCU/USB_N: track 2.70 -> 5.80 mm
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Other:
- board size 72 x 40.8 mm -> 73 x 40.8 mm
- board text added: "Nick Coombe (www.quizque.ca) Rev. B"
- board text removed: "Nick Coombe (www.quizque.ca) Rev. A"

Commit message: Stargazer PCB print update
Other:
- board text removed: "PCB3D_BR_main"
- board text removed: "PCB3D_TL_main"
